File: hardware/layouts/coldproff/coldproff.kicad_pcb (KiCad board)
At the start: 2 copper layers, 85 x 55 mm, 18 parts, among them J1 SWD 5p 1.27mm, U1 TPS61221DCKR, U2 STM32L010F4P6, U3 BC65PB-04-STD, U4 TMP117MAIDRCR, U5 ST25DV64KC6

Commit message: Update BC65 schematic symbol, footprint, and PCB for Rev B
- Create Quectel_BC65.pretty/Quectel_BC65.kicad_mod (identical LCC-58
  package to BC66, same pad positions and numbering 1-58)
- Update BC65 lib_symbols: pin numbers now match actual BC65 hardware
  (42/43=VBAT, 1/10/27/36=GND, 7=PWRKEY, 15=RESET_N, 16=NETLIGHT,
  17=MAIN_TXD, 18=MAIN_RXD, 34=GND_ANT, 35=ANT_RF)
- Pin names updated: STATUS→NETLIGHT, UART_TX→MAIN_TXD,
  UART_RX→MAIN_RXD, ANT_MAIN→ANT_RF, VCC1/2→VBAT1/2
- Footprint reference changed from Quectel_BC65:BC65-LCC to
  Quectel_BC65:Quectel_BC65 (in schematic and PCB)
- PCB footprint descriptor updated from BC66 to BC65 with correct
  datasheet URL; 3D model reuses BC66 step (identical physical package)

Co-Authored-By: Claude Sonnet 4.6 <noreply@anthropic.com>
Parts:
- U3: footprint Quectel_BC66 -> Quectel_BC65:Quectel_BC65
Changed lines of the file:
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@@
 		)
 	)
-	(footprint "Quectel_BC66"
+	(footprint "Quectel_BC65:Quectel_BC65"
 		(layer "F.Cu")
 		(at 17 27 90)
-		(descr "GSM NB-IoT module, 15.8x17.7x2mm, https://www.quectel.com/UploadImage/Downlad/Quectel_BC66_Hardware_Design_V1.1.pdf")
-		(tags "GSM NB-IoT Module BC66 M66")
+		(descr "NB-IoT module BC65PB-04-STD, 15.8x17.7x2mm LCC-58, https://www.quectel.com/content/uploads/2024/02/Quectel_BC65_Hardware_Design_V1.0-1.pdf")
+		(tags "NB-IoT BC65 LCC-58")
 		(property "Reference" "U3"
 			(at 0 -12.6 90)
